File: esp12-board.sch (KiCad schematic (older format))
At the start: 21 parts

Commit message: wip
Parts:
- removed P?: USB_B, symbol USB_B
- added P1: USB_OTG, Connect:USB_Mini-B, symbol USB_OTG
- BAT1: footprint (none) -> Pin_Headers:Pin_Header_Angled_1x02
- D1: renamed from D?; footprint (none) -> LEDs:LED_0805
- D2, D3, D4: renamed from D?; footprint (none) -> Diodes_SMD:SMA_Standard
- JP1, JP2: renamed from JP?; footprint (none) -> Pin_Headers:Pin_Header_Straight_1x02
- P2, P5: renamed from P?; footprint (none) -> Pin_Headers:Pin_Header_Straight_1x05
- P3: renamed from P?; footprint (none) -> Pin_Headers:Pin_Header_Straight_1x06
- P4: renamed from P?; footprint (none) -> Pin_Headers:Pin_Header_Angled_1x07
- R1, R2, R3, R4, R5: renamed from R?; footprint (none) -> Resistors_SMD:R_1206_HandSoldering
- SW1, SW2: renamed from SW?; footprint (none) -> Buttons_Switches_SMD:SW_SPST_EVQPE1
- U1: renamed from U?; footprint (none) -> TO_SOT_Packages_SMD:SOT-23-5
- U2: renamed from U?; footprint (none) -> ESP8266:ESP-12E
Connections:
- net GND: now also P1.5 (GND)
- net USBVCC: now also D1.2 (A), D2.2 (A), U1.4 (VDD), P1.1 (VBUS)
- net at BAT1.1 (P1), U1.3 (VBAT): now also D4.2 (A)
- no-connect marks 3 -> 4
